Commit message: body hight 재정의 및 각도로 재정의

File: ros2_ws/src/adom_description/urdf/adom_vehicle.urdf.xacro (robot description, xacro)
@@ -10,8 +10,21 @@
   <xacro:arg name="zed_y" default="0.0"/>
   <xacro:arg name="zed_z" default="0.24"/>
-  <xacro:arg name="zed_pitch" default="-0.1745"/>
+  <xacro:arg name="zed_pitch_deg" default="-9.9981"/>
   <xacro:arg name="gnss_x" default="0.0"/>
   <xacro:arg name="gnss_y" default="0.0"/>
   <xacro:arg name="gnss_z" default="0.30"/>
+  <!-- Expose command-line xacro arguments as expression variables. -->
+  <xacro:property name="wheelbase" value="$(arg wheelbase)"/>
+  <xacro:property name="track_width" value="$(arg track_width)"/>
+  <xacro:property name="body_length" value="$(arg body_length)"/>
+  <xacro:property name="body_width" value="$(arg body_width)"/>
+  <xacro:property name="body_height" value="$(arg body_height)"/>
+  <xacro:property name="zed_x" value="$(arg zed_x)"/>
+  <xacro:property name="zed_y" value="$(arg zed_y)"/>
+  <xacro:property name="zed_z" value="$(arg zed_z)"/>
+  <xacro:property name="zed_pitch_deg" value="$(arg zed_pitch_deg)"/>
+  <xacro:property name="gnss_x" value="$(arg gnss_x)"/>
+  <xacro:property name="gnss_y" value="$(arg gnss_y)"/>
+  <xacro:property name="gnss_z" value="$(arg gnss_z)"/>
   <link name="base_footprint"/>
   <link name="base_link">
@@ -31,5 +44,6 @@
   <link name="zed_camera_link"/>
   <joint name="zed_mount_joint" type="fixed">
-    <origin xyz="${zed_x} ${zed_y} ${zed_z}" rpy="0 ${zed_pitch} 0"/>
+    <!-- URDF rpy requires radians, so convert the degree-facing mount setting here. -->
+    <origin xyz="${zed_x} ${zed_y} ${zed_z}" rpy="0 ${zed_pitch_deg * pi / 180.0} 0"/>
     <parent link="base_link"/><child link="zed_camera_link"/>
   </joint>
